File: hardware/ModuLED_inicial/ModuLED_inicial.kicad_pcb (KiCad board)
At the start: 2 copper layers, 3 parts, among them U1 1088AS

Commit message: Primera Placa
Diseño de la primera placa para esta matriz, hecha para que tenga alimentación por batería con un regulador y los pines para sacar loscables que conecten a las entradas y salidas de los modulos. Despues se desglosó en filas y columnas los modulos para mas comodidad al conectar
Parts:
- added 100uF1: C_Polarized, Capacitor_THT:CP_Radial_D8.0mm_P2.50mm, F.Cu at (39.9, 43.7)
- added C1: 100 nF, Capacitor_THT:C_Disc_D3.4mm_W2.1mm_P2.50mm, F.Cu at (37.3, 51.9)
- added C2: 100nF, Capacitor_THT:C_Disc_D3.4mm_W2.1mm_P2.50mm, F.Cu at (34.8, 64.2)
- added C4: 100 uF, Capacitor_THT:CP_Radial_D8.0mm_P2.50mm, F.Cu at (34.8, 71.6)
- added Columnas2: Conn_01x08_Pin, Connector_PinSocket_2.54mm:PinSocket_1x08_P2.54mm_Vertical, F.Cu at (140.2, 33.7)
- added Columnas3: Conn_01x08_Pin, Connector_PinSocket_2.54mm:PinSocket_1x08_P2.54mm_Vertical, F.Cu at (221.3, 33.7)
- added Filas2: Conn_01x08_Pin, Connector_PinSocket_2.54mm:PinSocket_1x08_P2.54mm_Vertical, F.Cu at (177.6, 42.4)
- added Filas3: Conn_01x08_Pin, Connector_PinSocket_2.54mm:PinSocket_1x08_P2.54mm_Vertical, F.Cu at (258.8, 42.7)
- added J1: Conn_01x02_Pin, Connector_PinHeader_2.54mm:PinHeader_1x02_P2.54mm_Vertical, F.Cu at (44.6, 70.4)
- added J2: Conn_01x02_Pin, Connector_Molex:Molex_KK-396_A-41791-0002_1x02_P3.96mm_Vertical, F.Cu at (40.0, 35.2)
- added Pines_para_Arduino1: Conn_01x02_Pin, Connector_PinHeader_2.54mm:PinHeader_1x02_P2.54mm_Vertical, F.Cu at (30.5, 35.2)
- added U2: 1088AS, lib_fp:LED_1088_Pin_Header, F.Cu at (150.2, 91.6)
- added U3: 1088AS, lib_fp:LED_1088_Pin_Header, F.Cu at (231.3, 91.4)
- added U4: LM7805_TO220, Package_TO_SOT_THT:TO-220-3_Vertical, F.Cu at (39.8, 58.0)
- moved Columnas1 95.6 mm to (57.8, 33.6), turned to 0 degrees
- moved Filas1 55.9 mm to (95.1, 42.4), turned to -90 degrees
- moved U1 41.0 mm to (67.8, 91.4)
Connections:
- net Colum_0 renamed Colum_0_M1
- net Colum_1 renamed Colum_1_M1
- net Colum_2 renamed Colum_2_M1
- net Colum_3 renamed Colum_3_M1
- net Colum_4 renamed Colum_4_M1
- net Colum_5 renamed Colum_5_M1
- net Colum_6 renamed Colum_6_M1
- net Colum_7 renamed Colum_7_M1
- net Fil_0 renamed Fil_0_M1
- net Fil_1 renamed Fil_1_M1
- net Fil_2 renamed Fil_2_M1
- net Fil_3 renamed Fil_3_M1
- net Fil_4 renamed Fil_4_M1
- net Fil_5 renamed Fil_5_M1
- net Fil_6 renamed Fil_6_M1
- net Fil_7 renamed Fil_7_M1
Routing:
- net Colum_4_M2: track 0.00 -> 95.6 mm
- net Colum_4_M3: track 0.00 -> 95.4 mm
- net Fil_2_M3: track 0.00 -> 82.1 mm
- net Fil_2_M2: track 0.00 -> 82.1 mm
- net Colum_4_M1: track 16.0 -> 95.4 mm
- net Colum_0_M1: track 0.00 -> 77.6 mm
- net Colum_0_M3: track 0.00 -> 77.6 mm
- net Colum_0_M2: track 0.00 -> 77.3 mm
- net Colum_2_M3: track 0.00 -> 77.1 mm
- net Colum_2_M2: track 0.00 -> 77.1 mm
- net Fil_5_M3: track 0.00 -> 69.7 mm
- net Fil_5_M2: track 0.00 -> 69.7 mm
- net Colum_1_M2: track 0.00 -> 62.4 mm
- net Colum_1_M3: track 0.00 -> 62.4 mm
- net Fil_2_M1: track 20.9 -> 82.1 mm
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- added copper zone on F.Cu, net (none)
- added copper zone on B.Cu, net GND
Other:
- board outline added: 249.5 x 70.6 mm
