File: hardware/ModuLED_inicial/ModuLED_inicial.kicad_sch (KiCad schematic)
At the start: 0 parts

Commit message: Primera Placa
Diseño de la primera placa para esta matriz, hecha para que tenga alimentación por batería con un regulador y los pines para sacar loscables que conecten a las entradas y salidas de los modulos. Despues se desglosó en filas y columnas los modulos para mas comodidad al conectar
Parts:
- added 100uF1: C_Polarized, Capacitor_THT:CP_Radial_D8.0mm_P2.50mm, symbol Device:C_Polarized
- added C1: 100 nF, Capacitor_THT:C_Disc_D3.4mm_W2.1mm_P2.50mm, symbol Device:C
- added C2: 100nF, Capacitor_THT:C_Disc_D3.4mm_W2.1mm_P2.50mm, symbol Device:C
- added C4: 100 uF, Capacitor_THT:CP_Radial_D8.0mm_P2.50mm, symbol Device:C_Polarized
- added Columnas1, Columnas2, Columnas3, Filas1, Filas2, Filas3: Conn_01x08_Pin, Connector_PinSocket_2.54mm:PinSocket_1x08_P2.54mm_Vertical, symbol Connector:Conn_01x08_Pin
- added J1, Pines_para_Arduino1: Conn_01x02_Pin, Connector_PinHeader_2.54mm:PinHeader_1x02_P2.54mm_Vertical, symbol Connector:Conn_01x02_Pin
- added J2: Conn_01x02_Pin, Connector_Molex:Molex_KK-396_A-41791-0002_1x02_P3.96mm_Vertical, symbol Connector:Conn_01x02_Pin
- added U1, U2, U3: 1088AS, lib_fp:LED_1088_Pin_Header, symbol LED_1088as:1088AS
- added U4: LM7805_TO220, Package_TO_SOT_THT:TO-220-3_Vertical, symbol Regulator_Linear:LM7805_TO220
Connections:
- new net +5V: C2.1, C4.1, J1.1 (Pin_1), U4.3 (VO)
- new net Colum_0_M1: Columnas1.8 (Pin_8), U1.13 (R1)
- new net Colum_0_M2: Columnas2.8 (Pin_8), U2.13 (R1)
- new net Colum_0_M3: Columnas3.8 (Pin_8), U3.13 (R1)
- new net Colum_1_M1: Columnas1.7 (Pin_7), U1.3 (R2)
- new net Colum_1_M2: Columnas2.7 (Pin_7), U2.3 (R2)
- new net Colum_1_M3: Columnas3.7 (Pin_7), U3.3 (R2)
- new net Colum_2_M1: Columnas1.6 (Pin_6), U1.4 (R3)
- new net Colum_2_M2: Columnas2.6 (Pin_6), U2.4 (R3)
- new net Colum_2_M3: Columnas3.6 (Pin_6), U3.4 (R3)
- new net Colum_3_M1: Columnas1.5 (Pin_5), U1.10 (R4)
- new net Colum_3_M2: Columnas2.5 (Pin_5), U2.10 (R4)
- new net Colum_3_M3: Columnas3.5 (Pin_5), U3.10 (R4)
- new net Colum_4_M1: Columnas1.4 (Pin_4), U1.6 (R5)
- new net Colum_4_M2: Columnas2.4 (Pin_4), U2.6 (R5)
- new net Colum_4_M3: Columnas3.4 (Pin_4), U3.6 (R5)
- new net Colum_5_M1: Columnas1.3 (Pin_3), U1.11 (R6)
- new net Colum_5_M2: Columnas2.3 (Pin_3), U2.11 (R6)
- new net Colum_5_M3: Columnas3.3 (Pin_3), U3.11 (R6)
- new net Colum_6_M1: Columnas1.2 (Pin_2), U1.15 (R7)
- new net Colum_6_M2: Columnas2.2 (Pin_2), U2.15 (R7)
- new net Colum_6_M3: Columnas3.2 (Pin_2), U3.15 (R7)
- new net Colum_7_M1: Columnas1.1 (Pin_1), U1.16 (R8)
- new net Colum_7_M2: Columnas2.1 (Pin_1), U2.16 (R8)
- new net Colum_7_M3: Columnas3.1 (Pin_1), U3.16 (R8)
- new net Fil_0_M1: Filas1.8 (Pin_8), U1.9 (C8)
- new net Fil_0_M2: Filas2.8 (Pin_8), U2.9 (C8)
- new net Fil_0_M3: Filas3.8 (Pin_8), U3.9 (C8)
- new net Fil_1_M1: Filas1.7 (Pin_7), U1.14 (C7)
- new net Fil_1_M2: Filas2.7 (Pin_7), U2.14 (C7)
- new net Fil_1_M3: Filas3.7 (Pin_7), U3.14 (C7)
- new net Fil_2_M1: Filas1.6 (Pin_6), U1.8 (C6)
- new net Fil_2_M2: Filas2.6 (Pin_6), U2.8 (C6)
- new net Fil_2_M3: Filas3.6 (Pin_6), U3.8 (C6)
- new net Fil_3_M1: Filas1.5 (Pin_5), U1.12 (C5)
- new net Fil_3_M2: Filas2.5 (Pin_5), U2.12 (C5)
- new net Fil_3_M3: Filas3.5 (Pin_5), U3.12 (C5)
- new net Fil_4_M1: Filas1.4 (Pin_4), U1.1 (C4)
- new net Fil_4_M2: Filas2.4 (Pin_4), U2.1 (C4)
- new net Fil_4_M3: Filas3.4 (Pin_4), U3.1 (C4)
- new net Fil_5_M1: Filas1.3 (Pin_3), U1.7 (C3)
- new net Fil_5_M2: Filas2.3 (Pin_3), U2.7 (C3)
- new net Fil_5_M3: Filas3.3 (Pin_3), U3.7 (C3)
- new net Fil_6_M1: Filas1.2 (Pin_2), U1.2 (C2)
- new net Fil_6_M2: Filas2.2 (Pin_2), U2.2 (C2)
- new net Fil_6_M3: Filas3.2 (Pin_2), U3.2 (C2)
- new net Fil_7_M1: Filas1.1 (Pin_1), U1.5 (C1)
- new net Fil_7_M2: Filas2.1 (Pin_1), U2.5 (C1)
- new net Fil_7_M3: Filas3.1 (Pin_1), U3.5 (C1)
- new net GND: 100uF1.2, C1.1, C2.2, C4.2, J1.2 (Pin_2), J2.2 (Pin_2), Pines_para_Arduino1.2 (Pin_2), U4.2 (GND)
- new net VCC: 100uF1.1, C1.2, J2.1 (Pin_1), Pines_para_Arduino1.1 (Pin_1), U4.1 (VI)
